File: radio-battery-replacement/radio-battery-replacement.kicad_pcb (KiCad board)
At the start: 2 copper layers, 43 x 100 mm, 0 parts

Commit message: version v0.1.0 and fab outputs
Parts:
- added J2: USB_C_Receptacle_PowerOnly_6P, Connector_USB:USB_C_Receptacle_GCT_USB4135-GF-A_6P_TopMnt_Horizontal, F.Cu at (111.5, 76.0)
- added R1: 5k1, Resistor_SMD:R_1206_3216Metric_Pad1.30x1.75mm_HandSolder, F.Cu at (123.0, 77.0)
- added R2: 5k1, Resistor_SMD:R_1206_3216Metric_Pad1.30x1.75mm_HandSolder, F.Cu at (123.0, 74.0)
Routing:
- net +5V: track 0.00 -> 66.7 mm, vias 0 -> 4
- net Net-(J2-CC2): track 0.00 -> 14.5 mm
- net Net-(J2-CC1): track 0.00 -> 13.9 mm
- net GND: vias 0 -> 23
- added copper zone on B.Cu, net +5V
- added copper zone on F.Cu, net +5V
- added copper zone on B.Cu, net GND
- added copper zone on F.Cu, net GND
Other:
- board size 43 x 100 mm -> 43 x 49.5 mm
- net class Default removed
- rule solder_mask_min_width: 0.25 -> 0.16
- board text added: "+VE"
- board text added: "RADIO BATTERY ADAPTER V0.1.0"
